File: DesignPower.kicad_sch (KiCad schematic)
At the start: 23 parts, among them J1 Conn_01x02_Pin, J2 Conn_02x08_Odd_Even, U1 TP4056, U2 DRV8837, U3 DRV8837

Commit message: added jumper for current and labels on schematic logic
Parts:
- added JP1: Jumper_2_Open, symbol Jumper:Jumper_2_Open
Connections:
- net B+: now also JP1.2 (B); no longer J1.2 (Pin_2)
- new net: J1.2 (Pin_2), JP1.1 (A)
Other:
- note added: "R prog limits the current that flows from the IC"
- note added: "These ICs do all the logic work to run the motors"
- note added: "This is where our current test will be conducted"
- note added: "This pad was grounded as it was not in use.Grounded to avoid floating pins."
- note removed: "ADD NOTES"
- moved on the sheet: C3, C4, C5, C6, TPBat2, U2, U3
